File: roborio_expansion_boards/dio_adapter.brd (EAGLE design)
At the start: 16.8 x 76.2 mm, 20 parts

Commit message: added capacitors to the power lines near each connector
Parts:
- added C1, C10, C2, C3, C4, C5, C6, C7, C8, C9: 0.1 uF, custom:0603
Connections:
- net N$1: now also C1.1
- net N$10: now also C8.1, U$13.1, U$3.1; no longer U$17.1, U$7.1
- net N$11: now also C4.2
- net N$13: now also C7.1, U$14.1, U$4.1; no longer U$16.1, U$6.1
- net N$14: now also C5.2
- net N$16: now also C6.1
- net N$17: now also C6.2
- net N$19: now also C5.1, U$16.1, U$6.1; no longer U$14.1, U$4.1
- net N$2: now also C1.2
- net N$20: now also C7.2
- net N$22: now also C4.1, U$17.1, U$7.1; no longer U$13.1, U$3.1
- net N$23: now also C8.2
- net N$25: now also C3.1, U$18.1, U$8.1; no longer U$12.1, U$2.1
- net N$26: now also C9.2
- net N$28: now also C2.1, U$19.1, U$9.1; no longer U$1.1, U$11.1
- net N$29: now also C10.2
- net N$4: now also C10.1, U$1.1, U$11.1; no longer U$19.1, U$9.1
- net N$5: now also C2.2
- net N$7: now also C9.1, U$12.1, U$2.1; no longer U$18.1, U$8.1
- net N$8: now also C3.2
Routing:
- net N$1: track 13.2 -> 15.3 mm
- net N$5: track 11.4 -> 13.4 mm
- net N$2: track 11.4 -> 13.4 mm
- net N$14: track 11.4 -> 13.4 mm
- net N$29: track 11.4 -> 13.4 mm
- net N$23: track 11.4 -> 13.4 mm
- net N$20: track 11.4 -> 13.4 mm
- net N$26: track 11.4 -> 13.4 mm
- net N$11: track 11.4 -> 13.4 mm
- net N$8: track 11.4 -> 13.4 mm
- net N$17: track 11.4 -> 13.4 mm
- net N$4: track 14.0 -> 15.3 mm
- net N$19: track 14.0 -> 15.3 mm
- net N$10: track 14.0 -> 15.3 mm
- net N$28: track 14.0 -> 15.3 mm
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