File: roborio_expansion_boards/analog_adapter.brd (EAGLE design)
At the start: 16.8 x 76.2 mm, 30 parts

Commit message: finish PCBs and generate Gerbers for Seeed
Parts:
- removed C10, C5, C6, C7, C8, C9: 0.1 uF, custom:0603
- removed U$1, U$2, U$3, U$4, U$5, U$6: 22-23-2031GENERIC, custom:PWM_1X3
- removed U$11, U$12, U$13, U$14, U$15, U$16: 22-23-2031, custom:22-23-2031
- moved C1 45.7 mm to (3.81, 24.4)
- moved C2 45.7 mm to (3.81, 16.8)
- moved C3 45.7 mm to (3.81, 9.21)
- moved C4 45.7 mm to (3.81, 1.59)
- moved U$10 45.7 mm to (5.08, 26.7)
- moved U$17 45.7 mm to (12.7, 3.81)
- moved U$18 45.7 mm to (12.7, 11.4)
- moved U$19 45.7 mm to (12.7, 19.1)
- moved U$20 45.7 mm to (12.7, 26.7)
- moved U$7 45.7 mm to (5.08, 3.81)
- moved U$8 45.7 mm to (5.08, 11.4)
- moved U$9 45.7 mm to (5.08, 19.1)
Connections:
- removed net N$10: C8.1, U$13.3, U$3.1
- removed net N$13: C7.1, U$14.3, U$4.1
- removed net N$14: C5.2, U$16.2, U$6.2
- removed net N$15: U$16.1, U$6.3
- removed net N$16: C6.1, U$15.3, U$5.1
- removed net N$17: C6.2, U$15.2, U$5.2
- removed net N$18: U$15.1, U$5.3
- removed net N$19: C5.1, U$16.3, U$6.1
- removed net N$20: C7.2, U$14.2, U$4.2
- removed net N$21: U$14.1, U$4.3
- removed net N$23: C8.2, U$13.2, U$3.2
- removed net N$24: U$13.1, U$3.3
- removed net N$26: C9.2, U$12.2, U$2.2
- removed net N$27: U$12.1, U$2.3
- removed net N$29: C10.2, U$1.2, U$11.2
- removed net N$30: U$1.3, U$11.1
- removed net N$4: C10.1, U$1.1, U$11.3
- removed net N$7: C9.1, U$12.3, U$2.1
Routing:
- net N$19: track 15.3 -> 0.00 mm
- net N$7: track 15.3 -> 0.00 mm
- net N$4: track 15.3 -> 0.00 mm
- net N$13: track 15.3 -> 0.00 mm
- net N$10: track 15.3 -> 0.00 mm
- net N$16: track 15.3 -> 0.00 mm
- net N$14: track 13.4 -> 0.00 mm
- net N$29: track 13.4 -> 0.00 mm
- net N$26: track 13.4 -> 0.00 mm
- net N$23: track 13.4 -> 0.00 mm
- net N$20: track 13.4 -> 0.00 mm
- net N$17: track 13.4 -> 0.00 mm
- net N$21: track 7.62 -> 0.00 mm
- net N$30: track 7.62 -> 0.00 mm
- net N$27: track 7.62 -> 0.00 mm
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Other:
- board size 16.8 x 76.2 mm -> 16.8 x 30.5 mm
- board text added: "FRC Team 971 Analog Connector Adapter 20140818"
- board text removed: "4"
- board text removed: "5"
- board text removed: "6"
- board text removed: "7"
- board text removed: "8"
- board text removed: "9"
- board text removed: "FRC Team 971 DIO Connector Adapter 20140818"
