File: roborio_expansion_boards/analog_adapter.sch (EAGLE design)
At the start: 30 parts

Commit message: finish PCBs and generate Gerbers for Seeed
Parts:
- removed C10, C5, C6, C7, C8, C9: 0.1 uF, custom:CAP0603
- removed U$1, U$2, U$3, U$4, U$5, U$6: 22-23-2031GENERIC, custom:22-23-2031GENERIC
- removed U$11, U$12, U$13, U$14, U$15, U$16: 22-23-2031, custom:22-23-2031
Connections:
- removed net N$10: C8.1, U$13.SIG, U$3.GND
- removed net N$13: C7.1, U$14.SIG, U$4.GND
- removed net N$14: C5.2, U$16.PWR, U$6.PWR
- removed net N$15: U$16.GND, U$6.SIG
- removed net N$16: C6.1, U$15.SIG, U$5.GND
- removed net N$17: C6.2, U$15.PWR, U$5.PWR
- removed net N$18: U$15.GND, U$5.SIG
- removed net N$19: C5.1, U$16.SIG, U$6.GND
- removed net N$20: C7.2, U$14.PWR, U$4.PWR
- removed net N$21: U$14.GND, U$4.SIG
- removed net N$23: C8.2, U$13.PWR, U$3.PWR
- removed net N$24: U$13.GND, U$3.SIG
- removed net N$26: C9.2, U$12.PWR, U$2.PWR
- removed net N$27: U$12.GND, U$2.SIG
- removed net N$29: C10.2, U$1.PWR, U$11.PWR
- removed net N$30: U$1.SIG, U$11.GND
- removed net N$4: C10.1, U$1.GND, U$11.SIG
- removed net N$7: C9.1, U$12.SIG, U$2.GND
Other:
- moved on the sheet: C1, C2, C3, C4, U$10, U$17, U$18, U$19, U$20, U$7, U$8, U$9
