File: roborio_expansion_boards/pwm_adapter.sch (EAGLE design)
At the start: 30 parts

Commit message: finish PCBs and generate Gerbers for Seeed
Connections:
- net N$1: now also U$20.GND; no longer U$20.SIG
- net N$10: now also U$13.GND; no longer U$13.SIG
- net N$12: now also U$17.SIG; no longer U$17.GND
- net N$13: now also U$14.GND; no longer U$14.SIG
- net N$15: now also U$16.SIG; no longer U$16.GND
- net N$16: now also U$15.GND; no longer U$15.SIG
- net N$18: now also U$15.SIG; no longer U$15.GND
- net N$19: now also U$16.GND; no longer U$16.SIG
- net N$21: now also U$14.SIG; no longer U$14.GND
- net N$22: now also U$17.GND; no longer U$17.SIG
- net N$24: now also U$13.SIG; no longer U$13.GND
- net N$25: now also U$18.GND; no longer U$18.SIG
- net N$27: now also U$12.SIG; no longer U$12.GND
- net N$28: now also U$19.GND; no longer U$19.SIG
- net N$3: now also U$20.SIG; no longer U$20.GND
- net N$30: now also U$11.SIG; no longer U$11.GND
- net N$4: now also U$11.GND; no longer U$11.SIG
- net N$6: now also U$19.SIG; no longer U$19.GND
- net N$7: now also U$12.GND; no longer U$12.SIG
- net N$9: now also U$18.SIG; no longer U$18.GND
